Commit message: 20200319

File: binpicking/urdf/binpicking_robot.urdf.xacro (robot description, xacro)
@@ -26,4 +26,9 @@
     kinematics_file="${load_yaml('$(arg kinematics_config)')}"
     />
+  <!-- bracket/beugel -->
+  <xacro:include filename="$(find binpicking_support)/beugel/urdf/Beugel.urdf.xacro" />
+  <xacro:beugel/>
+  <!-- camera -->
+  <xacro:include filename="$(find realsense2_description)/urdf/_d435.urdf.xacro" />
   <link name="world" />
   <link name="baseplate_link">
@@ -61,3 +66,33 @@
     <origin xyz="0.0 0.0 0.01" rpy="0.0 0.0 0.0"/>
   </joint>
+  <link name="beugel_base_position"/>
+  <!-- tool0 to beugel_base_position -->
+  <!-- cahnge these valuse to place the beugel on the right position -->
+  <joint name="beugel_base_position_to_tool0" type="fixed">
+    <parent link="tool0" />
+    <child link="beugel_base_position" />
+    <origin xyz="0.0 0.00 0.01" rpy="${pi/2} 0.0 0.0"/> <!-- deze waardes zijn ook nogniet geheel juist-->
+  </joint>
+  <joint name="beugel_link_to_beugel_base_position" type="fixed">
+    <parent link="beugel_base_position" />
+    <child link="beugel_link" />
+    <origin xyz="0.0 0.0 0.0" rpy="0.0 0.0 0.0"/>
+  </joint>
+  <link name="beugel_camera_position"/>
+  <!-- beugel_base_position to beugel_camera_position -->
+  <joint name="beugel_to_beugel_base_position" type="fixed">
+    <parent link="beugel_link" />
+    <child link="beugel_camera_position" />
+    <origin xyz="0.0 -0.0049 0.0507" rpy="0.0 ${pi/6} -${pi/2}"/>
+  </joint>
+ <link name="camera_mouniting_holes"/>
+ <joint name="camera_mouniting_holes_to_beugel_camera_position" type="fixed">
+    <parent link="beugel_camera_position" />
+    <child link="camera_mouniting_holes" />
+    <origin xyz="-0.006 0.0 -0.006" rpy="0.0 0.0 ${pi}"/> <!-- deze waardes zijn nog niet geheel juist, natrekken bij mechanische tekeningen camera-->
+ </joint>
+  <!-- camera_to robot -->
+  <xacro:sensor_d435 parent="camera_mouniting_holes" use_nominal_extrinsics="true">
+    <origin xyz="0.0 0 0" rpy="0.0 0 0"/>
+  </xacro:sensor_d435>
 </robot>

Commit message: 20200319-3

File: binpicking/urdf/binpicking_robot.urdf.xacro (robot description, xacro)
@@ -72,5 +72,5 @@
     <parent link="tool0" />
     <child link="beugel_base_position" />
-    <origin xyz="0.0 0.00 0.01" rpy="${pi/2} 0.0 0.0"/> <!-- deze waardes zijn ook nogniet geheel juist-->
+    <origin xyz="0.0 0.00 0.01" rpy="${pi/2} 0 ${pi}"/> <!-- deze waardes zijn ook nogniet geheel juist-->
   </joint>
   <joint name="beugel_link_to_beugel_base_position" type="fixed">

Commit message: 2020413

File: binpicking/urdf/binpicking_robot.urdf.xacro (robot description, xacro)
@@ -31,4 +31,7 @@
   <!-- camera -->
   <xacro:include filename="$(find realsense2_description)/urdf/_d435.urdf.xacro" />
+  <!-- Vacuum Gripper -->
+  <xacro:include filename="$(find binpicking_support)/vacuum_gripper/urdf/vacuum_gripper.urdf.xacro" />
+  <xacro:vacuum_gripper_urdf prefix="gripper_" joint_prefix="suction_cup"/>
   <link name="world" />
   <link name="baseplate_link">
@@ -72,5 +75,5 @@
     <parent link="tool0" />
     <child link="beugel_base_position" />
-    <origin xyz="0.0 0.00 0.01" rpy="${pi/2} 0 ${pi}"/> <!-- deze waardes zijn ook nogniet geheel juist-->
+    <origin xyz="0.0 0.00 0.009" rpy="${pi/2} 0 ${pi}"/> <!-- deze waardes zijn ook nogniet geheel juist-->
   </joint>
   <joint name="beugel_link_to_beugel_base_position" type="fixed">
@@ -96,3 +99,8 @@
     <origin xyz="0.0 0 0" rpy="0.0 0 0"/>
   </xacro:sensor_d435>
+  <joint name="gripper_to_tool1" type="fixed">
+    <parent link="tool0" />
+    <child link="gripper_base_link" />
+    <origin xyz="0.00 0.00 0.005" rpy="0.0 0.0 0.0"/>
+  </joint>
 </robot>

Commit message: 20200617

File: binpicking/urdf/binpicking_robot.urdf.xacro (robot description, xacro)
@@ -32,6 +32,6 @@
   <xacro:include filename="$(find realsense2_description)/urdf/_d435.urdf.xacro" />
   <!-- Vacuum Gripper -->
-  <xacro:include filename="$(find binpicking_support)/vacuum_gripper/urdf/vacuum_gripper.urdf.xacro" />
-  <xacro:vacuum_gripper_urdf prefix="gripper_" joint_prefix="suction_cup"/>
+  <xacro:include filename="$(find binpicking_support)/epick_gripper/urdf/epick_gripper.urdf.xacro" />
+  <xacro:epick_gripper_urdf prefix="epick_gripper_"/>
   <link name="world" />
   <link name="baseplate_link">
@@ -99,4 +99,5 @@
     <origin xyz="0.0 0 0" rpy="0.0 0 0"/>
   </xacro:sensor_d435>
+<!--
   <joint name="gripper_to_tool1" type="fixed">
     <parent link="tool0" />
@@ -104,3 +105,9 @@
     <origin xyz="0.00 0.00 0.005" rpy="0.0 0.0 0.0"/>
   </joint>
+-->
+<joint name="beugel_to_epick_gripper" type ="fixed">
+    <parent link="tool0" />
+    <child link="epick_gripper_base_link" />
+    <origin xyz="0.00072798 0.089658 -0.0080751" rpy="0.0 0.0 0.0"/>
+  </joint>
 </robot>

Commit message: 20200707

File: binpicking/urdf/binpicking_robot.urdf.xacro (robot description, xacro)
@@ -109,5 +109,10 @@
     <parent link="tool0" />
     <child link="epick_gripper_base_link" />
-    <origin xyz="0.00072798 0.089658 -0.0080751" rpy="0.0 0.0 0.0"/>
+<!--
+    <origin xyz="0.00072798 0.089658 ${-0.0080751 + 0.011}" rpy="0.0 0.0 0.0"/>
+    <origin xyz="0.089658 0.00072798 -0.0080751 + 0.011}" rpy="0.0 0.0 ${pi}"/>
+    <origin xyz="${0.00072798 + 0.089658} 0.089658 ${-0.0080751 + 0.011}" rpy="0.0 0.0 ${pi}"/>
+-->
+    <origin xyz="0.00072798 -0.089658 ${-0.0080751 + 0.011}" rpy="0.0 0.0 ${pi}"/>
   </joint>
 </robot>
